File: component_tester.kicad_pcb (KiCad board)
At the start: 2 copper layers, 71 parts, among them IC1 ATMEGA16U2, IC2 ATMEGA328P-A, P1 USB_OTG, P10 BO_PC5, P11 ICSP_prog_328p, P12 CONN_01X01, P13 Device Under Test, P2 BATTERY_CONNECTOR, P3 Voltage_for_zener, P4 ICSP_prog_16u2, P5 BO_PC7, P6 BO_PD0, P7 BO_PD1, P8 BO_PC4, P9 BO_PC6, Q1 TRANSISTOR_NPN_2N2222_KSP222A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, SW1 SWITCH_DPDT_GROUNDED_BODY, SW2 DO_MEASUREMENT, SW3 CONNECT_CAP, U1 NCP1117ST50T3G, U2 XF2L-2625-1A, U3 CDSOT23-SRV05-4, U4 LT1004, Y1 8MHz, Y2 16MHz

Commit message: PCB drawn
Parts:
- removed C12: 100n, Capacitors_SMD:C_0805_HandSoldering
- removed the D5 at (78.4, 105.4)
- removed the D6 at (221.7, 31.6)
- added D3: D, TO_SOT_Packages_SMD:SOT-23, F.Cu at (112.8, 63.0)
- added D7: P6KE6V8A, TO_SOT_Packages_SMD:SOT-23, F.Cu at (185.7, 54.4)
- added F1: FUSE, Resistors_SMD:R_0805_HandSoldering, F.Cu at (109.5, 41.2)
- added F2: FUSE, Resistors_SMD:R_0805_HandSoldering, F.Cu at (105.9, 63.2)
- added P12: BO_PD2, Pin_Headers:Pin_Header_Straight_1x01, F.Cu at (166.4, 34.3)
- added P13: BO_PD3, Pin_Headers:Pin_Header_Straight_1x01, F.Cu at (163.8, 34.3)
- added P14: BO_PD4, Pin_Headers:Pin_Header_Straight_1x01, F.Cu at (161.3, 34.3)
- added P15: BO_PD5, Pin_Headers:Pin_Header_Straight_1x01, F.Cu at (168.9, 64.1)
- added P16: BO_PD6, Pin_Headers:Pin_Header_Straight_1x01, F.Cu at (171.4, 64.1)
- D1, D2: footprint Diodes_SMD:SOD-323 -> TO_SOT_Packages_SMD:SOT-23
- D4: value D -> ZENER; footprint Diodes_SMD:SOD-323 -> TO_SOT_Packages_SMD:SOT-23
- SW1: value SWITCH_DPDT_GROUNDED_BODY -> ON-OFF switch
- moved C3 126.7 mm to (129.4, 40.0), turned to 90 degrees
- moved R19 126.1 mm to (170.6, 35.7), turned to 270 degrees
- moved R15 125.7 mm to (155.0, 40.2), turned to 180 degrees
- moved R1 121.6 mm to (156.1, 33.5)
- moved R2 116.6 mm to (156.1, 35.6), turned to 180 degrees
- moved R17 115.9 mm to (149.0, 40.2), turned to 180 degrees
- moved R6 107.0 mm to (136.1, 43.7)
- moved R8 105.6 mm to (148.5, 56.0), turned to 270 degrees
- moved R10 105.2 mm to (169.5, 55.8)
- moved C2 102.3 mm to (115.9, 49.6), turned to 180 degrees
- moved C13 102.3 mm to (177.5, 44.8)
- moved C7 101.9 mm to (105.8, 35.0), turned to 90 degrees
- moved C5 100.6 mm to (105.8, 39.8), turned to 270 degrees
- moved R7 97.9 mm to (120.4, 55.4), turned to 270 degrees
- moved R9 97.7 mm to (150.7, 56.0), turned to 270 degrees
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- renumbered C6 to C11, C17 to C16, C18 to C17, C19 to C18, C16 to C19, C8 to C4, C4 to C5, C5 to C6, C11 to C8, D3 to D5, D7 to D6, P12 to P17, P13 to P18, R15 to R14, R14 to R15, R17 to R16, R16 to R17, R6 to R3, R3 to R4, R4 to R5, R5 to R6, U4 to U3, U3 to U4
Connections:
- C16 pad 1: Net-(C17-Pad1) -> GND
- C17 pad 1: Net-(C17-Pad1) -> GND
- C5 pad 1: Net-(C4-Pad1) -> Batt_Switch
- C8 pad 1: Battery_input -> Net-(C8-Pad1)
- C8 pad 2: Net-(C11-Pad2) (its old number) -> GND
- D4 pad 1: Battery_input -> Net-(C8-Pad1)
- D4 pad 2: Net-(D4-Pad2) -> GND
- IC1 pad 10: /control-niet_data-wel -> /lcd_reset-niet
- IC1 pad 12: /lcd_reset-niet -> /control-niet_data-wel
- L1 pad 2: Net-(D4-Pad2) -> Net-(D3-Pad2)
- Q1 pad 3: Net-(D4-Pad2) -> Net-(D3-Pad2)
- R1 pad 1: Battery_input -> Batt_Switch
- SW1 pad 1: 5Volt_328 -> Net-(F1-Pad1)
- SW1 pad 2: /USB_Vcc -> /Volt_reg_5v
- SW1 pad 3: /Volt_reg_5v -> /USB_Vcc
- SW1 pad 4: Net-(C4-Pad1) -> Batt_Switch
- SW1 pad 5: Net-(SW1-Pad5) -> Battery_input
- SW1 pad 6: Battery_input -> Net-(SW1-Pad6)
- U1 pad 3: Net-(C4-Pad1) -> Batt_Switch
Routing:
- net GND: track 0.00 -> 156.2 mm, vias 0 -> 36
- net 5Volt_328: track 0.00 -> 154.2 mm, vias 0 -> 8
- net 3Volt_16u: track 0.00 -> 77.3 mm, vias 0 -> 4
- net /USB_Vcc: track 0.00 -> 76.7 mm, vias 0 -> 2
- net /DUT1: track 0.00 -> 63.7 mm, vias 0 -> 2
- net Batt_Switch: track 0.00 -> 61.5 mm, vias 0 -> 2
- net UART_16u_TO_328: track 0.00 -> 55.4 mm, vias 0 -> 2
- net UART_328_TO_16u: track 0.00 -> 49.3 mm, vias 0 -> 2
- net /DUT3: track 0.00 -> 48.0 mm, vias 0 -> 3
- net /DUT2: track 0.00 -> 42.5 mm, vias 0 -> 3
- net Battery_input: track 0.00 -> 42.1 mm
- net /CHARGER_SWITCHING: track 0.00 -> 32.7 mm, vias 0 -> 2
- net /RESET_328: track 0.00 -> 32.2 mm, vias 0 -> 1
- net Net-(IC2-Pad11): track 0.00 -> 29.7 mm, vias 0 -> 1
- net Net-(IC1-Pad29): track 0.00 -> 29.3 mm, vias 0 -> 2
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- added copper zone on B.Cu, net GND
- added copper zone on F.Cu, net GND
Other:
- board outline added: 93 x 34 mm
- board text added: "2016-06-17"
- board text added: "ETGD component tester"
